Commit message: Uncomment hull link and joint definitions in URDF

File: src/ripc_description/urdf/ripc_usv.urdf.xacro (robot description, xacro)
@@ -20,5 +20,5 @@
   <!-- Hull -->
   <!-- Assume non-zero diagnoal values because of the hull's shape and mass distribution -->
-  <!-- <link name="hull">
+  <link name="hull">
     <inertial>
       <origin xyz="0 0 -0.15" rpy="0 0 0"/>
@@ -28,5 +28,4 @@
                izz="42"/>
     </inertial> -->
-    <!--  -->
     <visual>
       <origin xyz="0.446 0 0.0127" rpy="0 0 1.5708"/>
@@ -46,5 +45,5 @@
     </collision> -->
   <!-- </link> -->
-  <!-- <joint name="base_to_hull" type="fixed">
+  <joint name="base_to_hull" type="fixed">
     <parent link="base_link"/>
     <child link="hull"/>
